Commit message: Updated URDF model with screwdriver

File: urdf/screwdriver_tool.xacro (robot description, xacro)
@@ -10,7 +10,7 @@
       <visual>
         <geometry>
-          <cylinder length="0.05" radius="0.02"/>
+          <cylinder length="0.06" radius="0.02"/>
         </geometry>
-        <origin rpy="0 0 0" xyz="0 0 0.0255"/>
+        <origin rpy="0 0 0" xyz="0 0 0.0305"/>
         <material name="black">
           <color rgba="0 0 0 1"/>
@@ -19,7 +19,7 @@
       <collision>
         <geometry>
-          <cylinder length="0.05" radius="0.02"/>
+          <cylinder length="0.06" radius="0.02"/>
         </geometry>
-        <origin rpy="0 0 0" xyz="0 0 0.0255"/>
+        <origin rpy="0 0 0" xyz="0 0 0.0305"/>
       </collision>
     </link>
@@ -27,12 +27,12 @@
       <parent link="${prefix}screwdriver_holder"/>
       <child link="${prefix}screwdriver"/>
-      <origin rpy="0 0 0" xyz="0 0 0"/>
+      <origin rpy="0 0 0" xyz="0 0 0.146"/>
     </joint>
     <link name="${prefix}screwdriver">
       <visual>
         <geometry>
-          <cylinder length="0.1" radius="0.01"/>
+          <cylinder length="0.126" radius="0.01"/>
         </geometry>
-        <origin rpy="0 0 0" xyz="0 0 0.0505"/>
+        <origin rpy="0 0 0" xyz="0 0 -0.0635"/>
         <material name="wood">
           <color rgba=".87 .72 .53 1"/>
@@ -41,7 +41,7 @@
       <collision>
         <geometry>
-          <cylinder length="0.1" radius="0.01"/>
+          <cylinder length="0.126" radius="0.01"/>
         </geometry>
-        <origin rpy="0 0 0" xyz="0 0 0.0505"/>
+        <origin rpy="0 0 0" xyz="0 0 -0.0635"/>
       </collision>
     </link>

File: urdf/ur3e_with_screwdriver_tool.xacro (robot description, xacro)
@@ -8,5 +8,8 @@
   <xacro:include filename="screwdriver_tool.xacro" />
   <!-- arm -->
-  <xacro:ur3e_robot prefix="" joint_limited="false"/>
+  <xacro:arg name="kinematics_config" default="$(find ur_e_description)/config/ur3e_default.yaml"/>
+  <xacro:ur3e_robot prefix="" joint_limited="false"
+    kinematics_file="${load_yaml('$(arg kinematics_config)')}"
+  />
   <!-- end-effector -->
   <xacro:screwdriver_tool prefix="" connected_to="tool0"/>

Commit message: Updated screwdriver model

File: urdf/screwdriver_tool.xacro (robot description, xacro)
@@ -27,12 +27,12 @@
       <parent link="${prefix}screwdriver_holder"/>
       <child link="${prefix}screwdriver"/>
-      <origin rpy="0 0 0" xyz="0 0 0.146"/>
+      <origin rpy="0 0 0" xyz="0 0 0.123"/>
     </joint>
     <link name="${prefix}screwdriver">
       <visual>
         <geometry>
-          <cylinder length="0.126" radius="0.01"/>
+          <cylinder length="0.123" radius="0.01"/>
         </geometry>
-        <origin rpy="0 0 0" xyz="0 0 -0.0635"/>
+        <origin rpy="0 0 0" xyz="0 0 -0.0616"/>
         <material name="wood">
           <color rgba=".87 .72 .53 1"/>
@@ -41,7 +41,7 @@
       <collision>
         <geometry>
-          <cylinder length="0.126" radius="0.01"/>
+          <cylinder length="0.123" radius="0.01"/>
         </geometry>
-        <origin rpy="0 0 0" xyz="0 0 -0.0635"/>
+        <origin rpy="0 0 0" xyz="0 0 -0.0616"/>
       </collision>
     </link>

Commit message: Adding int screw trigger and including screwdriver in KDL chain

File: urdf/screwdriver_tool.xacro (robot description, xacro)
@@ -5,5 +5,5 @@
       <parent link="${connected_to}"/>
       <child link="${prefix}screwdriver_holder"/>
-      <origin rpy="0 0 0" xyz="0 0 0"/>
+      <origin rpy="0 ${-pi/2.0} ${-pi}" xyz="0 0 0"/>
     </joint>
     <link name="${prefix}screwdriver_holder">

File: urdf/ur3e_with_screwdriver_tool.xacro (robot description, xacro)
@@ -13,5 +13,5 @@
   />
   <!-- end-effector -->
-  <xacro:screwdriver_tool prefix="" connected_to="tool0"/>
+  <xacro:screwdriver_tool prefix="" connected_to="ee_link"/>
   <link name="world" />
   <joint name="world_joint" type="fixed">

Commit message: Last fixes to screwdriver in URDF

File: urdf/screwdriver_tool.xacro (robot description, xacro)
@@ -5,5 +5,5 @@
       <parent link="${connected_to}"/>
       <child link="${prefix}screwdriver_holder"/>
-      <origin rpy="0 ${-pi/2.0} ${-pi}" xyz="0 0 0"/>
+      <origin rpy="0 0 0" xyz="0 0 0"/>
     </joint>
     <link name="${prefix}screwdriver_holder">
@@ -12,5 +12,5 @@
           <cylinder length="0.06" radius="0.02"/>
         </geometry>
-        <origin rpy="0 0 0" xyz="0 0 0.0305"/>
+        <origin rpy="0 ${-pi/2.0} 0" xyz="0.0305 0 0"/>
         <material name="black">
           <color rgba="0 0 0 1"/>
@@ -21,5 +21,5 @@
           <cylinder length="0.06" radius="0.02"/>
         </geometry>
-        <origin rpy="0 0 0" xyz="0 0 0.0305"/>
+        <origin rpy="0 ${-pi/2.0} 0" xyz="0.0305 0 0"/>
       </collision>
     </link>
@@ -27,5 +27,5 @@
       <parent link="${prefix}screwdriver_holder"/>
       <child link="${prefix}screwdriver"/>
-      <origin rpy="0 0 0" xyz="0 0 0.123"/>
+      <origin rpy="0 0 0" xyz="0.123 0 0"/>
     </joint>
     <link name="${prefix}screwdriver">
@@ -34,5 +34,5 @@
           <cylinder length="0.123" radius="0.01"/>
         </geometry>
-        <origin rpy="0 0 0" xyz="0 0 -0.0616"/>
+        <origin rpy="0 ${-pi/2.0} 0" xyz="-0.0616 0 0"/>
         <material name="wood">
           <color rgba=".87 .72 .53 1"/>
@@ -43,5 +43,5 @@
           <cylinder length="0.123" radius="0.01"/>
         </geometry>
-        <origin rpy="0 0 0" xyz="0 0 -0.0616"/>
+        <origin rpy="0 ${-pi/2.0} 0" xyz="-0.0616 0 0"/>
       </collision>
     </link>
